File: PCB/pcb pulpo.sch (KiCad schematic (older format))
At the start: 71 parts, among them J1 fan1, J10 fan9, J11 fan10, J12 izq, J13 dcha, J14 inf, J15 Entrada 12V, J2 fan2, J3 fan3, J4 fan4, J5 fan5, J6 direct output, J7 fan6, J8 fan7, J9 fan8, U1 Teensy3.0, U2 LM7805_TO220

Commit message: Esquema y PCB en versión release 1
Parts:
- renumbered J15 to J0, J11 to J10, J6 to J11, J7 to J6, J8 to J7, J9 to J8, J10 to J9
Connections:
- net pin10: now also MOS_7.1 (G), R7.1, R_LED_7.1; no longer MOS_10.1 (G), R10.1, R_LED_10.1
- net pin7: now also MOS_10.1 (G), R10.1, R_LED_10.1; no longer MOS_7.1 (G), R7.1, R_LED_7.1
- net pin8: now also MOS_9.1 (G), R9.1, R_LED_9.1; no longer MOS_8.1 (G), R8.1, R_LED_8.1
- net pin9: now also MOS_8.1 (G), R8.1, R_LED_8.1; no longer MOS_9.1 (G), R9.1, R_LED_9.1
Changed lines of the file:
@@
 Title "HinchOSHWI"
 Date ""
-Rev "0.1"
+Rev "1"
 Comp "FotomatOSHWDem TEAM"
 Comment1 "Iraisy C. - Milo B. - Pablo. G"
@@
 $EndDescr
 $Comp
-L Connector:Screw_Terminal_01x02 J15
+L Connector:Screw_Terminal_01x02 J0
 U 1 1 5BC8F2A8
 P 7600 1250
-F 0 "J15" V 7473 1330 50  0000 L CNN
+F 0 "J0" V 7473 1330 50  0000 L CNN
 F 1 "Entrada 12V" V 7750 950 50  0000 L CNN
 F 2 "teensy:conector pablo pulpo hinchoshwi" H 7600 1250 50  0001 C CNN
@@
 $EndComp
 $Comp
-L Connector:Screw_Terminal_01x02 J7
+L Connector:Screw_Terminal_01x02 J6
 U 1 1 5C79A0EE
 P 5000 1000
-F 0 "J7" V 5100 750 50  0001 L CNN
+F 0 "J6" V 5100 750 50  0001 L CNN
 F 1 "fan6" V 5100 900 50  0000 L CNN
 F 2 "TerminalBlock:TerminalBlock_bornier-2_P5.08mm" H 5000 1000 50  0001 C CNN
@@
 $EndComp
 $Comp
-L Connector:Screw_Terminal_01x02 J8
+L Connector:Screw_Terminal_01x02 J7
 U 1 1 5C79A13C
 P 5000 2200
-F 0 "J8" V 5100 1950 50  0001 L CNN
+F 0 "J7" V 5100 1950 50  0001 L CNN
 F 1 "fan7" V 5100 2100 50  0000 L CNN
 F 2 "TerminalBlock:TerminalBlock_bornier-2_P5.08mm" H 5000 2200 50  0001 C CNN
@@
 $EndComp
 Text GLabel 3100 1800 0    50   Input ~ 0
-pin7
+pin10
 Wire Wire Line
 	3400 2650 3400 2550
@@
 $EndComp
 $Comp
-L Connector:Screw_Terminal_01x02 J9
+L Connector:Screw_Terminal_01x02 J8
 U 1 1 5C79A18B
 P 5000 3400
-F 0 "J9" V 5100 3150 50  0001 L CNN
+F 0 "J8" V 5100 3150 50  0001 L CNN
 F 1 "fan8" V 5100 3300 50  0000 L CNN
 F 2 "TerminalBlock:TerminalBlock_bornier-2_P5.08mm" H 5000 3400 50  0001 C CNN
@@
 $EndComp
 Text GLabel 3100 3000 0    50   Input ~ 0
-pin8
+pin9
 Wire Wire Line
 	3400 3850 3400 3750
@@
 $EndComp
 $Comp
-L Connector:Screw_Terminal_01x02 J10
+L Connector:Screw_Terminal_01x02 J9
 U 1 1 5C79A1D9
 P 5000 4600
-F 0 "J10" V 5100 4350 50  0001 L CNN
+F 0 "J9" V 5100 4350 50  0001 L CNN
 F 1 "fan9" V 5100 4500 50  0000 L CNN
 F 2 "TerminalBlock:TerminalBlock_bornier-2_P5.08mm" H 5000 4600 50  0001 C CNN
@@
 $EndComp
 Text GLabel 3100 4200 0    50   Input ~ 0
-pin9
+pin8
 Wire Wire Line
 	3400 5050 3400 4950
@@
 $EndComp
 $Comp
-L Connector:Screw_Terminal_01x02 J11
+L Connector:Screw_Terminal_01x02 J10
 U 1 1 5C79A228
 P 5000 5800
-F 0 "J11" V 5100 5550 50  0001 L CNN
+F 0 "J10" V 5100 5550 50  0001 L CNN
 F 1 "fan10" V 5100 5650 50  0000 L CNN
 F 2 "TerminalBlock:TerminalBlock_bornier-2_P5.08mm" H 5000 5800 50  0001 C CNN
@@
 $EndComp
 Text GLabel 3100 5400 0    50   Input ~ 0
-pin10
+pin7
 Wire Wire Line
 	3400 6250 3400 6150
@@
 Connection ~ 7450 3850
 $Comp
-L Connector:Screw_Terminal_01x02 J6
+L Connector:Screw_Terminal_01x02 J11
 U 1 1 5C0F288D
 P 2950 6900
-F 0 "J6" V 3050 6650 50  0001 L CNN
+F 0 "J11" V 3050 6650 50  0001 L CNN
 F 1 "direct output" V 3050 6600 50  0000 L CNN
 F 2 "TerminalBlock:TerminalBlock_bornier-2_P5.08mm" H 2950 6900 50  0001 C CNN
